File: KiCad Schematics/Mnt Circuits.kicad_sch (KiCad schematic)
At the start: 8 parts

Commit message: kicad schematics finalised
Parts:
- added SW1, SW2: SW_Push, symbol Switch:SW_Push
- MAX4466: value ~ -> StethoSense
- R1, R2, R3: value 100 ohm -> 630 ohm
- stretch sensor: renamed from R4
Connections:
- net GND: now also SW1.2, SW2.2
- net at MS2.27 (EN): now also SW2.1
- net at MS1.27 (EN): now also SW1.1
